File: Lab6/lab6Schema/lab6Schema.kicad_sch (KiCad schematic)
At the start: 9 parts, among them SW0 S0, SW1 S1, U1 74HC04, U2 74LS10, U3 74LS10

Commit message: update
Parts:
- removed unit 4 of U2
Changed lines of the file:
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@@
-	)
-	(symbol
-		(lib_id "74xx:74LS10")
-		(at 231.14 135.89 0)
-		(unit 4)
-		(exclude_from_sim no)
-		(in_bom yes)
-		(on_board yes)
-		(dnp no)
-		(fields_autoplaced yes)
-		(property "Reference" "U2"
-			(at 237.49 134.6199 0)
-			(effects
-				(font
-					(size 1.27 1.27)
-				)
-				(justify left)
-			)
-		)
-		(property "Value" "74LS10"
-			(at 237.49 137.1599 0)
-			(effects
-				(font
-					(size 1.27 1.27)
-				)
-				(justify left)
-			)
-		)
-		(property "Footprint" ""
-			(at 231.14 135.89 0)
-			(effects
-				(font
-					(size 1.27 1.27)
-				)
-				(hide yes)
-			)
-		)
-		(property "Datasheet" "http://www.ti.com/lit/gpn/sn74LS10"
-			(at 231.14 135.89 0)
-			(effects
-				(font
-					(size 1.27 1.27)
-				)
-				(hide yes)
-			)
-		)
-		(property "Description" "Triple 3-input NAND"
-			(at 231.14 135.89 0)
-			(effects
-				(font
-					(size 1.27 1.27)
-				)
-				(hide yes)
-			)
-		)
-		(pin "1"
-		)
-		(pin "7"
-		)
-		(pin "13"
-		)
-		(pin "8"
-		)
-		(pin "2"
-		)
-		(pin "6"
-		)
-		(pin "12"
-		)
-		(pin "4"
-		)
-		(pin "3"
-		)
-		(pin "10"
-		)
-		(pin "5"
-		)
-		(pin "9"
-		)
-		(pin "11"
-		)
-		(pin "14"
-		)
-		(instances
-			(project ""
-				(path "/4af3e3e9-c1e2-49d8-9fb7-b34eb0cb3c2e"
-					(reference "U2")
-					(unit 4)
-				)
-			)
-		)
 	)
 	(symbol
